Commit message: add forgotten files

File: robbie_description/urdf/rob_inmoov.xacro (robot description, xacro)
@@ -314,5 +314,5 @@
     	<origin xyz="-0.045 -0.145 0.105" rpy="0 0 0" />
         <axis xyz="1 0 0" />
-        <limit lower="-1.34" upper="0" effort="10" velocity="0" />
+        <limit lower="-1.34" upper="0.1" effort="10" velocity="0" />
 	</joint>
 <joint name="right_arm_lift_joint" type="revolute">
@@ -328,5 +328,5 @@
     	<origin xyz="0 0 -0.065" rpy="0 0 0" />
         <axis xyz="0 0 -1" />
-        <limit lower="-2.61" upper="0" effort="10" velocity="0" />
+        <limit lower="-3.14" upper="0.2" effort="10" velocity="0" />
 	</joint>
 <joint name="right_elbow_link" type="fixed">
@@ -412,5 +412,5 @@
     	<origin xyz="-0.045 0.145 0.105" rpy="0 0 0" />
         <axis xyz="-1 0 0" />
-        <limit lower="-1.34" upper="0" effort="10" velocity="0" />
+        <limit lower="-1.34" upper="0.1" effort="10" velocity="0" />
 	</joint>
 <joint name="left_arm_lift_joint" type="revolute">
@@ -426,5 +426,5 @@
     	<origin xyz="0 0.06 -0.055" rpy="0 0 0" />
         <axis xyz="0 0 -1" />
-        <limit lower="0" upper="2.61" effort="10" velocity="0" />
+        <limit lower="0.2" upper="3.14" effort="10" velocity="0" />
 	</joint>
 <joint name="left_elbow_link" type="fixed">

Commit message: add firmware files

File: robbie_description/urdf/rob_inmoov.xacro (robot description, xacro)
@@ -258,6 +258,36 @@
       </collision>
     </link>
-    <xacro:my_cylinder name="camera_link" l="0.035" r="0.008" xyz="0 0 0" rpy="0 1.57 0" mass="0.1" material="Gazebo/Grey">		<xacro:grey1 />
+    <xacro:my_cylinder name="camera_link" l="0.035" r="0.01" xyz="0 0 0" rpy="0 1.57 0" mass="0.1" material="Gazebo/Grey">
+      <xacro:grey1 />
 	</xacro:my_cylinder>
+<!-- virtal joints-->
+<link name="right_gripper_link">
+    <visual>
+      <origin rpy="0 0 0" xyz="0.05 0 0"/>
+      <geometry>
+        <box size="0.001 0.001 0.001"/>
+      </geometry>
+    </visual>
+    <collision>
+      <origin rpy="0 0 0" xyz="0.05 0 0"/>
+      <geometry>
+        <box size="0.001 0.001 0.001"/>
+      </geometry>
+    </collision>
+  </link>
+<link name="left_gripper_link">
+    <visual>
+      <origin rpy="0 0 0" xyz="-0.05 0 0"/>
+      <geometry>
+        <box size="0.001 0.001 0.001"/>
+      </geometry>
+    </visual>
+    <collision>
+      <origin rpy="0 0 0" xyz="-0.05 0 0"/>
+      <geometry>
+        <box size="0.001 0.001 0.001"/>
+      </geometry>
+    </collision>
+  </link>
 <!-- ##############################   joints ##################333333-->
 <joint name="base_footprint_joint" type="fixed">
@@ -297,5 +327,5 @@
     	<origin xyz="0.1 0 0.275" rpy="0 0 0" />
         <axis xyz="0 0 1" />
-        <limit lower="-0.26" upper="0.26" effort="10" velocity="0" />
+        <limit lower="-0.8" upper="0.8" effort="10" velocity="0" />
 	</joint>
   <joint name="torso_link" type="fixed">
@@ -386,4 +416,9 @@
     	<origin xyz="0.0 0.02 0.02" rpy="-1.57 0 1.57" />
 	</joint>
+  <joint name="right_gripper_joint" type="fixed">
+    <origin rpy="-1.570795 0 1.570795" xyz="0 0.06 0.01"/>
+    <parent link="gripper_bracket_f3"/>
+    <child link="right_gripper_link"/>
+  </joint>
 <!-- gripper_joint-->
    <joint name="right_arm_gripper_joint" type="revolute">
@@ -491,5 +526,5 @@
     	<parent link="left_wrist_tilt_bracket_f2" />
     	<child link="left_gripper_bracket_f3" />
-    	<origin xyz="0.0 0.035 0.0" rpy="0 1.57 0" />
+    	<origin xyz="0.0 0.035 0.0" rpy="0 0 0" />
 	</joint>
    <joint name="left_arm_gripper_servo" type="fixed">
@@ -498,4 +533,9 @@
     	<origin xyz="0.0 0.02 -0.02" rpy="0 3.14 0" />
 	</joint>
+  <joint name="left_gripper_joint" type="fixed">
+    <origin rpy="1.570795 0 1.570795" xyz="0 0.06 -0.01"/>
+    <parent link="left_gripper_bracket_f3"/>
+    <child link="left_gripper_link"/>
+  </joint>
   <!-- left gripper_joint-->
    <joint name="left_arm_gripper_joint" type="revolute"> <!--revolute-->
