Commit message: Upgrade to ROS Indigo

File: robbie_description/urdf/rob_inmoov.xacro (robot description, xacro)
@@ -10,5 +10,5 @@
     <property name="MESH_EXT" value="stl"/>
     <xacro:include filename="$(find robbie_description)/urdf/robbie_hardware.xacro" />
-<xacro:my_box name="base_link" lwh="0.41 0.35 0.06" xyz="0 0 .135" rpy="0 0 0" mass="0.1" material="Gazebo/FlatBlack">
+<xacro:my_box name="base_link" lwh="0.41 0.35 0.064" xyz="0 0 -0.032" rpy="0 0 0" mass="0.1" material="Gazebo/FlatBlack">
 	        <xacro:gold />
         </xacro:my_box>
@@ -34,5 +34,5 @@
 		<xacro:grey1 />
 	</xacro:my_cylinder>
-  <xacro:my_cylinder name="deck_link" l="0.520" r="0.175" xyz="0.1 0 0" rpy="0 0 0" mass="0.2" material="Gazebo/grey">
+  <xacro:my_cylinder name="deck_link" l="0.520" r="0.175" xyz="0 0 -0.26" rpy="0 0 0" mass="0.2" material="Gazebo/grey">
 			<xacro:black />
 		</xacro:my_cylinder>
@@ -47,5 +47,5 @@
       </geometry>
          <xacro:black/>
-      <origin rpy="0 0 -1.57" xyz="0 0 0"/>
+      <origin rpy="0 0 -1.57" xyz="0.04 0 -0.15"/>
     </visual>
   </link>
@@ -56,5 +56,5 @@
       </geometry>
          <xacro:gold/>
-      <origin rpy="0 0 1.57" xyz="0 0 0"/>
+      <origin rpy="0 0 1.57" xyz="0 0 -0.085"/>
     </visual>
   </link>
@@ -75,5 +75,5 @@
       </geometry>
        <xacro:black />
-      <origin rpy="0 0 1.57" xyz="-0.025 0 0.01"/>
+      <origin rpy="-1.57 0 1.57" xyz="-0.01 0 -0.025"/>
     </visual>
   </link>
@@ -84,5 +84,5 @@
       </geometry>
        <xacro:black/>
-      <origin rpy="0 1.57 0" xyz="0 0 0"/>
+      <origin rpy="0 0 0" xyz="0 0 0"/>
     </visual>
   </link>
@@ -93,5 +93,5 @@
       </geometry>
        <xacro:gold/>
-      <origin rpy="0 3.14 0" xyz="0 0 0"/>
+      <origin rpy="0 1.57 0" xyz="-0.19 0 0"/>
     </visual>
   </link>
@@ -102,5 +102,5 @@
       </geometry>
        <xacro:gold />
-      <origin rpy="3.14 0 0" xyz="0.025 -0.05 0.03"/>
+      <origin rpy="0 0 3.14" xyz="-0.025 -0.055 -0.02"/>
     </visual>
   </link>
@@ -111,21 +111,21 @@
       </geometry>
         <xacro:gold />
-      <origin rpy="0 -1.57 0" xyz="0 0 0"/>
+      <origin rpy="0 1.57 0" xyz="-0.23 0 0"/>
     </visual></link>
-  <!-- wrist_pan_ joint-->
-  <xacro:ax12 name="wrist_pan_servo" xyz="0 0 0" rpy="0 0 0" />
-  <xacro:F3_bracket name="wrist_pan_servo_bracket_f3" xyz="0 0.005 0" rpy="1.57 0 0" />
- <!-- <xacro:F3_bracket name="wrist_pan_servo_bracket2_f3" xyz="0 0 0" rpy="0 -1.57 0" />-->
+  <!-- wrist_yaw_ joint-->
+  <xacro:ax12 name="wrist_yaw_servo" xyz="0 0 0" rpy="-1.57 0 -1.57" />
+  <xacro:F3_bracket name="wrist_yaw_servo_bracket_f3" xyz="0 0.005 0" rpy="1.57 0 -1.57" />
+   <xacro:F2_bracket name="right_wrist_yaw_bracket_f2" xyz="0 0 0" rpy="-1.57 0 -1.57" />
   <!-- wrist_tilt joint-->
-  <xacro:ax12 name="wrist_tilt_servo" xyz="-0.04 0.05 0" rpy="-1.57 0 0" />
-  <xacro:F2_bracket name="wrist_tilt_bracket_f2" xyz="0 0 0" rpy="0 1.57 0" /><!--here-->
- <xacro:F3_bracket name="gripper_bracket_f3" xyz="0 0 0" rpy="1.57 1.57 0" />
+  <xacro:ax12 name="wrist_tilt_servo" xyz="0 0 0" rpy="0 -1.57 0" />
+  <xacro:F2_bracket name="wrist_tilt_bracket_f2" xyz="0 0 0" rpy="0 -1.57 0" /><!--here-->
+ <xacro:F3_bracket name="gripper_bracket_f3" xyz="0 0 0" rpy="1.57 0 -1.57" />
 <!-- Gripper_joint-->
   <xacro:ax12 name="gripper_servo" xyz="0 0 0" rpy="1.57 0 0" />
-  <xacro:F2_bracket name="gripper_bracket_f2" xyz="0 0 0" rpy="0 0 1.57" />
-  <xacro:my_box name="right_finger_link" lwh="-0.08 0.005 0.035" xyz="0 0 0" rpy="1.57 0 1.57" mass="0.1" material="Gazebo/FlatBlack">
+  <xacro:F2_bracket name="gripper_bracket_f2" xyz="0 0 0" rpy="1.57 0 0" />
+  <xacro:my_box name="right_finger_link" lwh="-0.08 0.005 0.035" xyz="-0.04 0 0" rpy="0 0 0" mass="0.1" material="Gazebo/FlatBlack">
 	        <xacro:blue1 />
         </xacro:my_box>
-  <xacro:my_box name="left_finger_link" lwh="0.08 0.005 0.035" xyz="0 0 0" rpy="1.57 0 1.57" mass="0.1" material="Gazebo/FlatBlack">
+  <xacro:my_box name="left_finger_link" lwh="0.08 0.005 0.035" xyz="-0.04 0 0" rpy="0 0 0" mass="0.1" material="Gazebo/FlatBlack">
 	        <xacro:grey3/>
         </xacro:my_box>
@@ -145,6 +145,6 @@
         <mesh filename="package://robbie_description/meshes/left_shoulder_assy.stl" scale="${M_SCALE} ${M_SCALE} ${M_SCALE}"/>
       </geometry>
-       <xacro:black />
-      <origin rpy="0 0 1.57" xyz="0 0 0"/>
+       <xacro:grey1 />
+      <origin rpy="-1.57 0 1.57" xyz="0 -0.06 0"/>
     </visual>
   </link>
@@ -155,5 +155,5 @@
       </geometry>
        <xacro:gold/>
-      <origin rpy="0 3.14 0" xyz="0 0 0"/>
+      <origin rpy="0 1.57 0" xyz="-0.19 0 0"/>
     </visual>
   </link>
@@ -164,5 +164,5 @@
       </geometry>
        <xacro:black/>
-      <origin rpy="0 1.57 0" xyz="0 0 0"/>
+      <origin rpy="0 0 0" xyz="0 0 0"/>
     </visual>
   </link>
@@ -173,5 +173,5 @@
       </geometry>
        <xacro:gold />
-      <origin rpy="3.14 0 0" xyz="0.025 -0.05 0.03"/>
+      <origin rpy="0 0 3.14" xyz="-0.025 -0.055 -0.02"/>
     </visual>
   </link>
@@ -182,25 +182,24 @@
       </geometry>
         <xacro:gold />
-      <origin rpy="0 -1.57 0" xyz="0 0 0"/>
+      <origin rpy="0 1.57 0" xyz="-0.23 0 0"/>
     </visual>
   </link>
  <!-- left_wrist_pan_ joint-->
-  <xacro:ax12 name="left_wrist_pan_servo" xyz="0 0 0" rpy="0 0 0" />
-  <xacro:F3_bracket name="left_wrist_pan_servo_bracket_f3" xyz="0 0.005 0" rpy="1.57 0 0" />
+  <xacro:F3_bracket name="left_wrist_pan_servo_bracket_f3" xyz="0 0.005 0" rpy="1.57 0 -1.57" />
  <!-- <xacro:F3_bracket name="left_wrist_pan_servo_bracket2_f3" xyz="0 0 0" rpy="0 -1.57 0" />-->
  <!-- left_wrist_yaw joint-->
-  <xacro:ax12 name="left_wrist_yaw_servo" xyz="-0.04 0.05 0" rpy="-1.57 0 0" />
-  <xacro:F2_bracket name="left_wrist_yaw_bracket_f2" xyz="0 0 0" rpy="-1.57 0 0" />
+  <xacro:ax12 name="left_wrist_yaw_servo" xyz="0.0 0 0" rpy="-1.57 0 -1.57" />
+  <xacro:F2_bracket name="left_wrist_yaw_bracket_f2" xyz="0 0 0" rpy="-1.57 0 -1.57" />
   <!-- left_wrist_tilt joint-->
-  <xacro:ax12 name="left_wrist_tilt_servo" xyz="0 0 0" rpy="1.57 1.57 0" />
-  <xacro:F2_bracket name="left_wrist_tilt_bracket_f2" xyz="0 0 0" rpy="1.57 1.57 0" />
- <xacro:F3_bracket name="left_gripper_bracket_f3" xyz="0 0 0" rpy="1.57 1.57 0" />
+  <xacro:ax12 name="left_wrist_tilt_servo" xyz="0 0 0" rpy="0 -1.57 0" />
+  <xacro:F2_bracket name="left_wrist_tilt_bracket_f2" xyz="0 0 0" rpy="0 -1.57 0" />
+ <xacro:F3_bracket name="left_gripper_bracket_f3" xyz="0 0 0" rpy="1.57 0 -1.57" />
 <!-- left_Gripper_joint-->
-  <xacro:ax12 name="left_gripper_servo" xyz="0 0 0" rpy="0 0 -1.57" />
-  <xacro:F2_bracket name="left_gripper_bracket_f2" xyz="0 0 0" rpy="0 0 1.57" />
-  <xacro:my_box name="left_right_finger_link" lwh="-0.08 0.005 0.035" xyz="0 0 0" rpy="1.57 0 1.57" mass="0.1" material="Gazebo/FlatBlack">
+  <xacro:ax12 name="left_gripper_servo" xyz="0 0 0" rpy="1.57 0 0" />
+  <xacro:F2_bracket name="left_gripper_bracket_f2" xyz="0 0 0" rpy="1.57 0 0" />
+  <xacro:my_box name="left_right_finger_link" lwh="-0.08 0.005 0.035" xyz="-0.04 0 0" rpy="0 0 0" mass="0.1" material="Gazebo/FlatBlack">
 	        <xacro:blue1 />
         </xacro:my_box>
-  <xacro:my_box name="left_left_finger_link" lwh="0.08 0.005 0.035" xyz="0 0 0" rpy="1.57 0 1.57" mass="0.1" material="Gazebo/FlatBlack">
+  <xacro:my_box name="left_left_finger_link" lwh="0.08 0.005 0.035" xyz="-0.04 0 0" rpy="0 0 0" mass="0.1" material="Gazebo/FlatBlack">
 	        <xacro:grey3/>
         </xacro:my_box>
@@ -294,30 +293,30 @@
     	<parent link="base_footprint" />
     	<child link="base_link" />
-    	<origin xyz="-0.1 0 0" rpy="0 0 0" />
+    	<origin xyz="-0.1 0 0.08" rpy="0 0 0" />
 	</joint>
 <joint name="base_link_joint" type="fixed">
     	<parent link="base_link" />
     	<child link="deck_link" />
-    	<origin xyz="-0.1 0 .36" rpy="0 0 0" />
+    	<origin xyz="0 0 0.51" rpy="0 0 0" />
 	</joint>
   <joint name="left_wheel_joint" type="fixed">
     	<parent link="base_link" />
     	<child link="left_wheel" />
-    	<origin xyz="0.1 -0.2 0.1" rpy="0 0 0" />
+    	<origin xyz="0.1 -0.2 -0.04" rpy="0 0 0" />
 	</joint>
   <joint name="right_wheel_joint" type="fixed">
     	<parent link="base_link" />
     	<child link="right_wheel" />
-    	<origin xyz="0.1 0.2 0.1" rpy="0 0 0" />
+    	<origin xyz="0.1 0.2 -0.04" rpy="0 0 0" />
 	</joint>
   <joint name="castor_wheel_joint_l" type="fixed">
     	<parent link="base_link" />
     	<child link="castor_wheel_l" />
-    	<origin xyz="-0.20 -0.13 0.05" rpy="0 0 0" />
+    	<origin xyz="-0.20 -0.13 -0.1" rpy="0 0 0" />
 	</joint>
   <joint name="castor_wheel_joint_r" type="fixed">
     	<parent link="base_link" />
     	<child link="castor_wheel_r" />
-    	<origin xyz="-0.20 0.13 0.05" rpy="0 0 0" />
+    	<origin xyz="-0.20 0.13 -0.1" rpy="0 0 0" />
 	</joint>
 <!--#################  Upper torso#############################-->
@@ -325,5 +324,5 @@
     	<parent link="deck_link" />
     	<child link="pan_link" />
-    	<origin xyz="0.1 0 0.275" rpy="0 0 0" />
+    	<origin xyz="0.0 0 0" rpy="0 0 0" />
         <axis xyz="0 0 1" />
         <limit lower="-1" upper="1" effort="10" velocity="0" />
@@ -332,15 +331,15 @@
     	<parent link="pan_link" />
     	<child link="upper_torso" />
-    	<origin xyz="0.05 0 0.26" rpy="0 0 0" />
+    	<origin xyz="0.0 0 0.47" rpy="0 0 0" />
 	</joint>
 <joint name="chest_link" type="fixed">
     	<parent link="upper_torso" />
     	<child link="upper_chest" />
-    	<origin xyz="0.02 0 0.03" rpy="0 0 0" />
+    	<origin xyz="0.065 0 -0.04" rpy="0 0 0" />
 	</joint>
 <joint name="right_arm_tilt_joint" type="revolute">
     	<parent link="upper_torso" />
     	<child link="right_shoulder_tilt" />
-    	<origin xyz="-0.045 -0.145 0.105" rpy="0 0 0" />
+    	<origin xyz="0 -0.14 -0.045" rpy="0 0 0" />
         <axis xyz="1 0 0" />
         <limit lower="-1.34" upper="0.1" effort="10" velocity="0" />
@@ -349,5 +348,5 @@
     	<parent link="right_shoulder_tilt" />
     	<child link="right_shoulder_lift" />
-    	<origin xyz="-0.0 -0.077 -0.04" rpy="0 -1.57 0" />
+    	<origin xyz="0 -0.078 -0.042" rpy="0 0 0" />
         <axis xyz="0 1 0" />
         <limit lower="-1.57" upper="1.57" effort="10" velocity="0" />
@@ -356,6 +355,6 @@
     	<parent link="right_shoulder_lift" />
     	<child link="right_shoulder_rotate" />
-    	<origin xyz="0 0 -0.065" rpy="0 0 0" />
-        <axis xyz="0 0 -1" />
+    	<origin xyz="0.255 0 0" rpy="0 0 0" />
+        <axis xyz="1 0 0" />
         <limit lower="-3.14" upper="0.2" effort="10" velocity="0" />
 	</joint>
@@ -363,10 +362,10 @@
     	<parent link="right_shoulder_rotate" />
     	<child link="right_elbow_link" />
-    	<origin xyz="0.01 0 -0.17" rpy="0 0 0" />
+    	<origin xyz="-0.01 0 0.01" rpy="0 0 0" />
         </joint>
 <joint name="right_arm_elbow_joint" type="revolute">
     <parent link="right_elbow_link"/>
     <child link="right_elbow"/>
-    <origin xyz="0.01 0.01 0.0" rpy="0 -1.57 0" />
+    <origin xyz="0.01 0.01 0.0" rpy="0 0 0" />
     <axis xyz="0 1 0" />
    <limit lower="-2.20" upper="0.1" effort="10" velocity="0" />
@@ -375,31 +374,38 @@
     <parent link="right_elbow"/>
     <child link="right_forearm_link"/>
-    <origin xyz="-0.08 -0.0 -0.0" rpy="1.57 0 0" />
+    <origin xyz="0.31 -0.0 -0.0" rpy="0 0 0" />
   </joint>
-  <!--right_arm_wrist_pan_joint-->
-  <joint name="right_arm_wrist_pan_bracket" type="fixed">
+  <!--right_arm_wrist_yaw_joint-->
+  <joint name="right_arm_wrist_yaw_bracket" type="fixed">
     	<parent link="right_forearm_link" />
-    	<child link="wrist_pan_servo" />
-    	<origin xyz="-0.21 0.0 0.0" rpy="0 0 1.57" />
-	</joint>
-  <joint name="right_arm_wrist_pan_joint" type="revolute">
-    	<parent link="wrist_pan_servo" />
-    	<child link="wrist_pan_servo_bracket_f3" />
-    	<origin xyz="0. 0.015 0.0" rpy="0 1.57 0" />
-        <axis xyz="0 1 0" />
+    	<child link="wrist_yaw_servo_bracket_f3" />
+    	<origin xyz="0.0 0.0 0.0" rpy="0 0 0" />
+	</joint>
+  <joint name="right_arm_wrist_yaw_bracket1" type="fixed">
+    	<parent link="wrist_yaw_servo_bracket_f3" />
+    	<child link="wrist_yaw_servo" />
+    	<origin xyz="0.04 0 0.0" rpy="0 0 0" />
+        <axis xyz="0 0 1" />
     	<limit lower="-2.61" upper="2.61" effort="10" velocity="0" />
       	<dynamics damping="0.0"/>
 	</joint>
-   <joint name="right_arm_wrist_tilt_bracket" type="fixed">
-    	<parent link="wrist_pan_servo_bracket_f3" />
+   <joint name="right_arm_wrist_yaw_joint" type="revolute">
+    	<parent link="wrist_yaw_servo" />
+    	<child link="right_wrist_yaw_bracket_f2" />
+    	<origin xyz="0.0 0 0.0" rpy="0 0 0" />
+        <axis xyz="0 0 1" />
+    	<limit lower="-2.61" upper="2.61" effort="10" velocity="0" />
+	</joint>
+<joint name="right_arm_wrist_tilt1_bracket" type="fixed">
+    	<parent link="right_wrist_yaw_bracket_f2" />
+    	<child link="wrist_tilt_bracket_f2" />
+    	<origin xyz="0.053 0 0.0" rpy="0 0 0" />
+        <axis xyz="0 0 1" />
+	</joint>
+<!--wrist_tilt_joint-->
+  <joint name="right_arm_wrist_tilt_joint" type="revolute">
+    	<parent link="wrist_tilt_bracket_f2" />
     	<child link="wrist_tilt_servo" />
-    	<origin xyz="0.04 0 0.0" rpy="0 0 0" />
-        <axis xyz="1 0 0" />
-	</joint>
-<!--wrist_tilt_joint-->
-  <joint name="right_arm_wrist_yaw_joint" type="revolute">
-    	<parent link="wrist_tilt_servo" />
-    	<child link="wrist_tilt_bracket_f2" />
-    	<origin xyz="-0.04 0.05 0" rpy="-1.57 0 1.57" />
+    	<origin xyz="0 0 0" rpy="0 0 0" />
         <axis xyz="0 1 0" />
     	<limit lower="-1.57" upper="1.57" effort="10" velocity="0" />
@@ -407,17 +413,17 @@
 	</joint>
   <joint name="right_arm_gripper_bracket" type="fixed">
-    	<parent link="wrist_tilt_bracket_f2" />
+    	<parent link="wrist_tilt_servo" />
     	<child link="gripper_bracket_f3" />
-    	<origin xyz="0.025 0.025 0.0" rpy="1.57 1.57 0" /><!--now-->
+    	<origin xyz="0.04 0 0.0" rpy="0 0 0" /><!--now-->
 	</joint>
    <joint name="right_arm_gripper_servo" type="fixed">
     	<parent link="gripper_bracket_f3" />
     	<child link="gripper_servo" />
-    	<origin xyz="0.0 0.02 0.02" rpy="-1.57 0 1.57" />
+    	<origin xyz="0.02 -0.015 0.0" rpy="0 0 0" />
 	</joint>
   <joint name="right_gripper_joint" type="fixed">
-    <origin rpy="-1.570795 0 1.570795" xyz="0 0.06 0.01"/>
     <parent link="gripper_bracket_f3"/>
     <child link="right_gripper_link"/>
+    <origin xyz="0.06 -0.01 0" rpy="0 0 0" />
   </joint>
 <!-- gripper_joint-->
@@ -425,7 +431,7 @@
     	<parent link="gripper_servo" />
     	<child link="gripper_bracket_f2" />
-    	<origin xyz="0 0.0 0.0" rpy="0 1.57 -1.57" />
-        <axis xyz="1 0 0" />
-    	<limit lower="-0.36" upper="0.28" effort="10" velocity="0" />
+    	<origin xyz="0 0.0 0.0" rpy="0 0 0" />
+        <axis xyz="0 0 1" />
+    	<limit lower="-0.1" upper="0.50" effort="10" velocity="0" />
       	<dynamics damping="0.0"/>
 	</joint>
@@ -433,5 +439,5 @@
     	<parent link="gripper_servo" />
     	<child link="left_finger_link" />
-    	<origin xyz="0.03 0.04 0.0" rpy="0 1.57 -1.57" />
+    	<origin xyz="0.08 0.04 0" rpy="0 0 0" />
 	</joint>
 <!-- moving finger   ############-->
@@ -439,5 +445,5 @@
     	<parent link="gripper_bracket_f2" />
     	<child link="right_finger_link" />
-    	<origin xyz="0 0.03 0.03" rpy="0 0 0" />
+    	<origin xyz="0.08 -0.03 0" rpy="0 0 0" />
 	</joint>
 <!--##########################        left arm             #############################-->
@@ -445,5 +451,5 @@
     	<parent link="upper_torso" />
     	<child link="left_shoulder_tilt" />
-    	<origin xyz="-0.045 0.145 0.105" rpy="0 0 0" />
+    	<origin xyz="0.003 0.142 -0.05" rpy="0 0 0" />
         <axis xyz="-1 0 0" />
         <limit lower="-1.34" upper="0.1" effort="10" velocity="0" />
@@ -452,5 +458,5 @@
     	<parent link="left_shoulder_tilt" />
     	<child link="left_shoulder_lift" />
-    	<origin xyz="0 0.02 -0.04" rpy="0 -1.57 0" />
+    	<origin xyz="0 0.08 -0.04" rpy="0 0 0" />
         <axis xyz="0 1 0" />
         <limit lower="-1.57" upper="1.57" effort="10" velocity="0" />
@@ -459,17 +465,17 @@
     	<parent link="left_shoulder_lift" />
     	<child link="left_shoulder_rotate" />
-    	<origin xyz="0 0.06 -0.055" rpy="0 0 0" />
-        <axis xyz="0 0 -1" />
-        <limit lower="0.2" upper="3.14" effort="10" velocity="0" />
+    	<origin xyz="0.24 0 0" rpy="0 0 0" />
+        <axis xyz="1 0 0" />
+        <limit lower="-0.2" upper="3.14" effort="10" velocity="0" />
 	</joint>
 <joint name="left_elbow_link" type="fixed">
     	<parent link="left_shoulder_rotate" />
     	<child link="left_elbow_link" />
-    	<origin xyz="0.01 0 -0.17" rpy="0 0 0" />
+    	<origin xyz="-0.01 0 0.008" rpy="0 0 0" />
 	</joint>
 <joint name="left_arm_elbow_joint" type="revolute">
     <parent link="left_elbow_link"/>
     <child link="left_elbow"/>
-    <origin xyz="0.01 0.01 0.0" rpy="0 -1.57 0" />
+    <origin xyz="0 0 0" rpy="0 -0 0" />
     <axis xyz="0 1 0" />
    <limit lower="-2.20" upper="0.17" effort="10" velocity="0" />
@@ -478,18 +484,10 @@
     <parent link="left_elbow"/>
     <child link="left_forearm_link"/>
-    <origin xyz="-0.08 -0.0 -0.0" rpy="1.57 0 0" />
+    <origin xyz="0.31 -0.0 -0.0" rpy="0 0 0" />
   </joint>
-    <!--left_arm_wrist_pan_joint-->
-  <joint name="left_arm_wrist_pan_bracket" type="fixed">
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
File: robbie_description/urdf/robbie_hardware.xacro (robot description, xacro)
@@ -88,5 +88,5 @@
 				<origin xyz="${xyz}" rpy="${rpy}" />
 				<geometry>
-					<mesh filename="package://robbie/meshes/ax12_box2.${MESH_EXT}" scale="${M_SCALE} ${M_SCALE} ${M_SCALE}"/>
+					<mesh filename="package://robbie_description/meshes/ax12_box2.${MESH_EXT}" scale="${M_SCALE} ${M_SCALE} ${M_SCALE}"/>
 				</geometry>
 				<xacro:ax12_color />
@@ -96,5 +96,5 @@
 				<geometry>
 					<!--<box size="0.032 0.038 0.05" />-->
-					<mesh filename="package://robbie/meshes/ax12_box2.${MESH_EXT}" scale="${M_SCALE} ${M_SCALE} ${M_SCALE}"/>
+					<mesh filename="package://robbie_description/meshes/ax12_box2.${MESH_EXT}" scale="${M_SCALE} ${M_SCALE} ${M_SCALE}"/>
 				</geometry>
              </collision>
@@ -108,12 +108,12 @@
 				<origin xyz="${xyz}" rpy="${rpy}" />
 				<geometry>
-          			<mesh filename="package://robbie/meshes/F2.${MESH_EXT}" scale="${M_SCALE} ${M_SCALE} ${M_SCALE}"/>
-				</geometry>
-				<xacro:bracket_color />
-             </visual>
-             <collision>
-				<origin xyz="${xyz}" rpy="${rpy}" />
-					<geometry>
-          				<mesh filename="package://robbie/meshes/F2.${MESH_EXT}" scale="${M_SCALE} ${M_SCALE} ${M_SCALE}"/>
+          			<mesh filename="package://robbie_description/meshes/F2.${MESH_EXT}" scale="${M_SCALE} ${M_SCALE} ${M_SCALE}"/>
+				</geometry>
+				<xacro:bracket_color />
+             </visual>
+             <collision>
+				<origin xyz="${xyz}" rpy="${rpy}" />
+					<geometry>
+          				<mesh filename="package://robbie_description/meshes/F2.${MESH_EXT}" scale="${M_SCALE} ${M_SCALE} ${M_SCALE}"/>
 					</geometry>
              </collision>
@@ -127,5 +127,5 @@
 				<origin xyz="${xyz}" rpy="${rpy}" />
 				<geometry>
-          			<mesh filename="package://robbie/meshes/F3.${MESH_EXT}" scale="${M_SCALE} ${M_SCALE} ${M_SCALE}"/>
+          			<mesh filename="package://robbie_description/meshes/F3.${MESH_EXT}" scale="${M_SCALE} ${M_SCALE} ${M_SCALE}"/>
 				</geometry><material name="grey1">
 			<color rgba="0.75 0.75 0.75 1.0"/>
@@ -136,5 +136,5 @@
 				<origin xyz="${xyz}" rpy="${rpy}" />
 					<geometry>
-          				<mesh filename="package://robbie/meshes/F3.${MESH_EXT}" scale="${M_SCALE} ${M_SCALE} ${M_SCALE}"/>
+          				<mesh filename="package://robbie_description/meshes/F3.${MESH_EXT}" scale="${M_SCALE} ${M_SCALE} ${M_SCALE}"/>
 					</geometry>
              </collision>
