Commit message: update
update

File: robbie_description/urdf/rob_inmoov.xacro (robot description, xacro)
@@ -6,4 +6,5 @@
        xmlns:xacro="http://ros.org/wiki/xacro"
 	   name="robbie">
+    <property name="PI" value="3.1415" />
     <property name="M_PI" value="3.14159"/>
     <property name="M_SCALE" value="0.001"/>
@@ -622,46 +623,60 @@
     	<origin xyz="0.2 0 0.33" rpy="0 0 0" />
 	</joint>
-  <joint name="kinect_depth_joint" type="fixed">
-      <origin xyz="0 0.018 0" rpy="0 0 0" />
-      <parent link="kinect_link" />
-      <child link="kinect_depth_frame" />
-    </joint>
-    <link name="kinect_depth_frame">
+<joint name="kinect_depth_joint" type="fixed">
+         <origin xyz="0 0.0125 0.015" rpy="0 0 0" />
+          <parent link="kinect_link" />
+          <child link="kinect_depth_frame" />
+      </joint>
+      <link name="kinect_depth_frame">
       <inertial>
-        <mass value="0.0001" />
-        <origin xyz="0 0 0" />
-        <inertia ixx="0.0001" ixy="0.0" ixz="0.0"
-                 iyy="0.0001" iyz="0.0"
-                 izz="0.0001" />
-      </inertial>
-    </link>
-    <joint name="kinect_depth_optical_joint" type="fixed">
-      <origin xyz="0 0 0" rpy="${-M_PI/2} 0 ${-M_PI/2}" />
-      <parent link="kinect_link" />
-      <child link="kinect_depth_optical_frame" />
-    </joint>
-    <link name="kinect_depth_optical_frame">
-      <inertial>
-        <mass value="0.0001" />
-        <origin xyz="0 0 0" />
-        <inertia ixx="0.0001" ixy="0.0" ixz="0.0"
-                 iyy="0.0001" iyz="0.0"
-                 izz="0.0001" />
-      </inertial>
-    </link>
-    <joint name="kinect_rgb_optical_joint" type="fixed">
-      <origin xyz="0 0 0" rpy="${-M_PI/2} 0 ${-M_PI/2}" />
-      <parent link="kinect_depth_optical_frame" />
-      <child link="kinect_rgb_optical_frame" />
-    </joint>
-    <link name="kinect_rgb_optical_frame">
-      <inertial>
-        <mass value="0.001" />
-        <origin xyz="0 0 0" />
-        <inertia ixx="0.0001" ixy="0.0" ixz="0.0"
-                 iyy="0.0001" iyz="0.0"
-                 izz="0.0001" />
-      </inertial>
-    </link>
+         <mass value="0.000001" />
+         <origin xyz="0 0 0" />
+         <inertia ixx="0.0001" ixy="0.0" ixz="0.0"
+            iyy="0.0001" iyz="0.0"
+            izz="0.0001" />
+         </inertial>
+      </link>
+      <joint name="kinect_depth_optical_joint" type="fixed">
+         <origin xyz="0 0 0" rpy="${-PI/2} 0 ${-PI/2}" />
+         <parent link="kinect_depth_frame" />
+         <child link="kinect_depth_optical_frame" />
+      </joint>
+      <link name="kinect_depth_optical_frame">
+         <inertial>
+            <mass value="0.000001" />
+            <origin xyz="0 0 0" />
+            <inertia ixx="0.0001" ixy="0.0" ixz="0.0"
+               iyy="0.0001" iyz="0.0"
+               izz="0.0001" />
+         </inertial>
+      </link>
+      <joint name="kinect_rgb_joint" type="fixed">
+         <origin xyz="0 -0.0125 0.015" rpy="0 0 0" />
+         <parent link="kinect_link" />
+         <child link="kinect_rgb_frame" />
+      </joint>
+      <link name="kinect_rgb_frame">
+         <inertial>
+         <mass value="0.000001" />
+         <origin xyz="0 0 0" />
+         <inertia ixx="0.0001" ixy="0.0" ixz="0.0"
+            iyy="0.0001" iyz="0.0"
+            izz="0.0001" />
+         </inertial>
+      </link>
+      <joint name="kinect_rgb_optical_joint" type="fixed">
+         <origin xyz="0 0 0" rpy="${-PI/2} 0 ${-PI/2}" />
+         <parent link="kinect_rgb_frame" />
+         <child link="kinect_rgb_optical_frame" />
+      </joint>
+      <link name="kinect_rgb_optical_frame">
+         <inertial>
+            <mass value="0.000001" />
+            <origin xyz="0 0 0" />
+            <inertia ixx="0.0001" ixy="0.0" ixz="0.0"
+               iyy="0.0001" iyz="0.0"
+               izz="0.0001" />
+         </inertial>
+      </link>
 <gazebo reference="robbie">
   	</gazebo>

Commit message: update

File: robbie_description/urdf/rob_inmoov.xacro (robot description, xacro)
@@ -219,10 +219,10 @@
    <visual>
       <geometry>
-        <mesh filename="package://robbie_description/meshes/head.stl" scale="${M_SCALE} ${M_SCALE} ${M_SCALE}"/>
+        <mesh filename="package://robbie_description/meshes/head1.stl" scale="${M_SCALE} ${M_SCALE} ${M_SCALE}"/>
       </geometry>
          <material name="gold">
 	  <color rgba="0.5 0.3 0 1.0"/>
 	</material>
-      <origin rpy="1.57 0 1.57" xyz="0 0 0"/>
+      <origin rpy="0 0 1.57" xyz="0 0 0"/>
     </visual>
   </link>
@@ -258,4 +258,26 @@
       </collision>
     </link>
+  <link name="head_cam_link">
+      <inertial>
+        <mass value="1.0" />
+        <origin xyz="0 0 0" />
+        <inertia ixx="1.0" ixy="0.0" ixz="0.0"
+                 iyy="1.0" iyz="0.0"
+                 izz="1.0" />
+      </inertial>
+      <visual>
+        <origin xyz=" 0 0 0 " rpy="0 0 0" />
+        <geometry>
+          <mesh filename="package://robbie_description/meshes/kinect.stl" scale="${M_SCALE} ${M_SCALE} ${M_SCALE}"/>
+        </geometry>
+        <xacro:ax12_color />
+      </visual>
+      <collision>
+        <origin xyz="0 0 0" rpy="0 0 0" />
+        <geometry>
+          <mesh filename="package://robbie_description/meshes/kinect.stl" scale="${M_SCALE} ${M_SCALE} ${M_SCALE}"/>
+          </geometry>
+      </collision>
+    </link>
     <xacro:my_cylinder name="camera_link" l="0.035" r="0.01" xyz="0 0 0" rpy="0 1.57 0" mass="0.1" material="Gazebo/Grey">
       <xacro:grey1 />
@@ -611,5 +633,5 @@
     	<parent link="head_base_link" />
     	<child link="head_link" />
-    	<origin xyz="-0.02 -0.097 -0.45" rpy="0 0 0" />
+    	<origin xyz="-0.02 -0.097 0" rpy="0 0 0" />
 	</joint>
    <joint name="camera_link" type="fixed">
@@ -679,4 +701,65 @@
          </inertial>
       </link>
+  <joint name="head_cam_joint" type="fixed">
+    	<parent link="head_link" />
+    	<child link="head_cam_link" />
+    	<origin xyz="0.15 0.11 0.13" rpy="0 0 0" />
+	</joint>
+<joint name="head_cam_depth_joint" type="fixed">
+         <origin xyz="0 0.0125 0.015" rpy="0 0 0" />
+          <parent link="head_cam_link" />
+          <child link="head_cam_depth_frame" />
+      </joint>
+      <link name="head_cam_depth_frame">
+      <inertial>
+         <mass value="0.000001" />
+         <origin xyz="0 0 0" />
+         <inertia ixx="0.0001" ixy="0.0" ixz="0.0"
+            iyy="0.0001" iyz="0.0"
+            izz="0.0001" />
+         </inertial>
+      </link>
+      <joint name="head_cam_depth_optical_joint" type="fixed">
+         <origin xyz="0 0 0" rpy="${-PI/2} 0 ${-PI/2}" />
+         <parent link="head_cam_depth_frame" />
+         <child link="head_cam_depth_optical_frame" />
+      </joint>
+      <link name="head_cam_depth_optical_frame">
+         <inertial>
+            <mass value="0.000001" />
+            <origin xyz="0 0 0" />
+            <inertia ixx="0.0001" ixy="0.0" ixz="0.0"
+               iyy="0.0001" iyz="0.0"
+               izz="0.0001" />
+         </inertial>
+      </link>
+      <joint name="head_cam_rgb_joint" type="fixed">
+         <origin xyz="0 -0.0125 0.015" rpy="0 0 0" />
+         <parent link="head_cam_link" />
+         <child link="head_cam_rgb_frame" />
+      </joint>
+      <link name="head_cam_rgb_frame">
+         <inertial>
+         <mass value="0.000001" />
+         <origin xyz="0 0 0" />
+         <inertia ixx="0.0001" ixy="0.0" ixz="0.0"
+            iyy="0.0001" iyz="0.0"
+            izz="0.0001" />
+         </inertial>
+      </link>
+      <joint name="head_cam_rgb_optical_joint" type="fixed">
+         <origin xyz="0 0 0" rpy="${-PI/2} 0 ${-PI/2}" />
+         <parent link="head_cam_rgb_frame" />
+         <child link="head_cam_rgb_optical_frame" />
+      </joint>
+      <link name="head_cam_rgb_optical_frame">
+         <inertial>
+            <mass value="0.000001" />
+            <origin xyz="0 0 0" />
+            <inertia ixx="0.0001" ixy="0.0" ixz="0.0"
+               iyy="0.0001" iyz="0.0"
+               izz="0.0001" />
+         </inertial>
+      </link>
 <gazebo reference="robbie">
   	</gazebo>
