Commit message: change AI

File: robbie_description/urdf/base2.xacro (robot description, xacro)
@@ -7,4 +7,23 @@
     <property name="MESH_EXT" value="stl"/>
     <xacro:include filename="$(find robbie_description)/urdf/robbie_hardware.xacro" />
+  <gazebo>
+  <plugin name="differential_drive_controller" filename="libgazebo_ros_diff_drive.so">
+    <alwaysOn>true</alwaysOn>
+    <updateRate>20</updateRate>
+    <leftJoint>base_link_left_wheel_joint</leftJoint>
+    <rightJoint>base_link_right_wheel_joint</rightJoint>
+    <wheelSeparation>0.430</wheelSeparation>
+    <wheelDiameter>0.2</wheelDiameter>
+    <torque>20</torque>
+    <commandTopic>cmd_vel</commandTopic>
+    <odometryTopic>odom</odometryTopic>
+    <odometryFrame>odom</odometryFrame>
+    <robotBaseFrame>base_footprint</robotBaseFrame>
+    <broadcastTF>true</broadcastTF>
+    <robotNamespace>robbie</robotNamespace>
+    <publishWheelTF>true</publishWheelTF>
+    <publishWheelJointState>true</publishWheelJointState>
+  </plugin>
+</gazebo>
    <!-- Import all Gazebo-customization elements, including Gazebo colors -->
   <xacro:include filename="$(find robbie_description)/urdf/robbie.gazebo" />
@@ -41,5 +60,5 @@
       <origin rpy="0 0 1.57" xyz=" 0.015 -0.175 -0"/>
     </visual>
-    <xacro:default_inertial mass="0.0001" />
+    <xacro:default_inertial mass="1.0" />
   </link>
  <xacro:my_cylinder name="pan_link" l="0.005" r="0.1" xyz="0.0 0 -0.02" rpy="0 0 0" mass="0.2" material="Gazebo/Grey">
@@ -85,10 +104,10 @@
     	<origin xyz="0 0 0.138" rpy="0 0 0" />
 	</joint>
-  <joint name="base_l_wheel_joint" type="fixed">
+  <joint name="base_link_left_wheel_joint" type="continuous">
     	<parent link="base_link" />
     	<child link="left_wheel" />
     	<origin xyz="0.1 -0.2 -0.04" rpy="0 0 0" />
 	</joint>
-  <joint name="base_r_wheel_joint" type="fixed">
+  <joint name="base_link_right_wheel_joint" type="continuous">
     	<parent link="base_link" />
     	<child link="right_wheel" />
@@ -128,4 +147,23 @@
     	<origin xyz="0.065 0 -0.04" rpy="0 0 0" />
 	</joint>
+<!-- Transmission is important to link the joints and the controller -->
+<transmission name="right_wheel_joint_trans">
+	<type>transmission_interface/SimpleTransmission</type>
+	<joint name="base_link_right_wheel_joint" />
+        <hardwareInterface>EffortJointInterface</hardwareInterface>
+<actuator name="base_link_right_wheel_joint_motor">
+	<hardwareInterface>EffortJointInterface</hardwareInterface>
+	<mechanicalReduction>1</mechanicalReduction>
+</actuator>
+</transmission>
+<transmission name="left_wheel_joint_trans">
+<type>transmission_interface/SimpleTransmission</type>
+<joint name="base_link_left_wheel_joint" />
+<hardwareInterface>EffortJointInterface</hardwareInterface>
+<actuator name="base_link_right_wheel_joint_motor">
+<hardwareInterface>EffortJointInterface</hardwareInterface>
+<mechanicalReduction>1</mechanicalReduction>
+</actuator>
+</transmission>
 <gazebo reference="robbie">
   	</gazebo>
