Commit message: daily update

File: robbie_description/urdf/rob_inmoov.urdf (robot description, URDF)
Before this commit: robot robbie, 55 links, 54 joints
Links:
- added link left_gripper_link; collision box size=0.001 0.001 0.001; visual box size=0.001 0.001 0.001
- added link right_gripper_link; collision box size=0.001 0.001 0.001; visual box size=0.001 0.001 0.001
Joints:
- added joint left_gripper_joint: type fixed, parent left_gripper_bracket_f3, child left_gripper_link, origin xyz=0 0.06 -0.01 rpy=1.570795 0 1.570795
- added joint right_gripper_joint: type fixed, parent gripper_bracket_f3, child right_gripper_link, origin xyz=0 0.06 0.01 rpy=-1.570795 0 1.570795
- joint left_arm_elbow_joint: limit lower=-2.00 upper=0.57 effort=10 velocity=0 -> lower=-2.20 upper=0.17 effort=10 velocity=0
- joint left_arm_gripper_bracket: parent left_wrist_tilt_bracket_f2 -> left_wrist_tilt_servo
- joint left_arm_wrist_pan_joint: origin xyz=0. 0.015 0.0 rpy=0 1.57 0 -> xyz=0. 0.015 0.0 rpy=0 0 0
- joint left_arm_wrist_tilt_joint: child left_wrist_tilt_bracket_f2 -> left_wrist_tilt_servo; origin xyz=-0.04 0.05 0 rpy=0 0 0 -> xyz=-0 -0.0 0 rpy=0 0 0; parent left_wrist_tilt_servo -> left_wrist_tilt_bracket_f2
- joint left_arm_wrist_yaw_bracket: axis (none) -> 1 0 0; child left_wrist_tilt_servo -> left_wrist_tilt_bracket_f2; limit (none) -> lower=-1.57 upper=1.57 effort=10 velocity=0; origin xyz=0.04 0 0.0 rpy=0 0 0 -> xyz=-0.0 0.052 0.0 rpy=0 0 0
- joint pan_joint: limit lower=-0.8 upper=0.8 effort=10 velocity=0 -> lower=-1 upper=1 effort=10 velocity=0
- joint right_arm_elbow_joint: limit lower=-2.00 upper=0.57 effort=10 velocity=0 -> lower=-2.20 upper=0.1 effort=10 velocity=0
- joint right_arm_wrist_pan_joint: origin xyz=0. 0.015 0.0 rpy=0 0 0 -> xyz=0. 0.015 0.0 rpy=0 1.57 0
- joint right_arm_wrist_yaw_joint: axis 0 0 1 -> 0 1 0

File: robbie_description/urdf/rob_inmoov.xacro (robot description, xacro)
@@ -193,5 +193,5 @@
   <xacro:F2_bracket name="left_wrist_yaw_bracket_f2" xyz="0 0 0" rpy="-1.57 0 0" />
   <!-- left_wrist_tilt joint-->
-  <xacro:ax12 name="left_wrist_tilt_servo" xyz="-0.04 0.05 0" rpy="1.57 1.57 0" />
+  <xacro:ax12 name="left_wrist_tilt_servo" xyz="0 0 0" rpy="1.57 1.57 0" />
   <xacro:F2_bracket name="left_wrist_tilt_bracket_f2" xyz="0 0 0" rpy="1.57 1.57 0" />
  <xacro:F3_bracket name="left_gripper_bracket_f3" xyz="0 0 0" rpy="1.57 1.57 0" />
@@ -327,5 +327,5 @@
     	<origin xyz="0.1 0 0.275" rpy="0 0 0" />
         <axis xyz="0 0 1" />
-        <limit lower="-0.8" upper="0.8" effort="10" velocity="0" />
+        <limit lower="-1" upper="1" effort="10" velocity="0" />
 	</joint>
   <joint name="torso_link" type="fixed">
@@ -370,5 +370,5 @@
     <origin xyz="0.01 0.01 0.0" rpy="0 -1.57 0" />
     <axis xyz="0 1 0" />
-   <limit lower="-2.00" upper="0.57" effort="10" velocity="0" />
+   <limit lower="-2.20" upper="0.1" effort="10" velocity="0" />
   </joint>
   <joint name="right_arm_forearm_link" type="fixed">
@@ -386,5 +386,5 @@
     	<parent link="wrist_pan_servo" />
     	<child link="wrist_pan_servo_bracket_f3" />
-    	<origin xyz="0. 0.015 0.0" rpy="0 0 0" />
+    	<origin xyz="0. 0.015 0.0" rpy="0 1.57 0" />
         <axis xyz="0 1 0" />
     	<limit lower="-2.61" upper="2.61" effort="10" velocity="0" />
@@ -402,5 +402,5 @@
     	<child link="wrist_tilt_bracket_f2" />
     	<origin xyz="-0.04 0.05 0" rpy="-1.57 0 1.57" />
-        <axis xyz="0 0 1" />
+        <axis xyz="0 1 0" />
     	<limit lower="-1.57" upper="1.57" effort="10" velocity="0" />
       	<dynamics damping="0.0"/>
@@ -473,5 +473,5 @@
     <origin xyz="0.01 0.01 0.0" rpy="0 -1.57 0" />
     <axis xyz="0 1 0" />
-   <limit lower="-2.00" upper="0.57" effort="10" velocity="0" />
+   <limit lower="-2.20" upper="0.17" effort="10" velocity="0" />
   </joint>
  <joint name="left_arm_forearm_link" type="fixed">
@@ -489,5 +489,5 @@
     	<parent link="left_wrist_pan_servo" />
     	<child link="left_wrist_pan_servo_bracket_f3" />
-    	<origin xyz="0. 0.015 0.0" rpy="0 1.57 0" />
+    	<origin xyz="0. 0.015 0.0" rpy="0 0 0" />
         <axis xyz="0 1 0" />
     	<limit lower="-2.61" upper="2.61" effort="10" velocity="0" />
@@ -511,12 +511,15 @@
   <joint name="left_arm_wrist_yaw_bracket" type="fixed">
     	<parent link="left_wrist_yaw_bracket_f2" />
-    	<child link="left_wrist_tilt_servo" />
-    	<origin xyz="0.04 0 0.0" rpy="0 0 0" />
+    	<child link="left_wrist_tilt_bracket_f2" />
+    	<origin xyz="-0.0 0.052 0.0" rpy="0 0 0" />
+        <axis xyz="1 0 0" />
+    	<limit lower="-1.57" upper="1.57" effort="10" velocity="0" />
+      	<dynamics damping="0.0"/>
         </joint>
   <!--wrist_tilt_joint-->
   <joint name="left_arm_wrist_tilt_joint" type="revolute"> <!--revolute-->
-    	<parent link="left_wrist_tilt_servo" />
-    	<child link="left_wrist_tilt_bracket_f2" />
-    	<origin xyz="-0.04 0.05 0" rpy="0 0 0" />
+    	<parent link="left_wrist_tilt_bracket_f2" />
+    	<child link="left_wrist_tilt_servo" />
+    	<origin xyz="-0 -0.0 0" rpy="0 0 0" />
         <axis xyz="1 0 0" />
     	<limit lower="-1.57" upper="1.57" effort="10" velocity="0" />
@@ -524,7 +527,7 @@
 	</joint>
   <joint name="left_arm_gripper_bracket" type="fixed">
-    	<parent link="left_wrist_tilt_bracket_f2" />
+    	<parent link="left_wrist_tilt_servo" />
     	<child link="left_gripper_bracket_f3" />
-    	<origin xyz="0.0 0.035 0.0" rpy="0 0 0" />
+    	<origin xyz="0.0 0.035 0.0" rpy="0 1.57 0" />
 	</joint>
    <joint name="left_arm_gripper_servo" type="fixed">

Commit message: add robbie_gazebo and control

File: robbie_description/urdf/rob_inmoov.urdf (robot description, URDF)
Before this commit: robot robbie, 57 links, 56 joints
Links:
- removed link camera_link
- removed link left_wrist_pan_servo
- removed link wrist_pan_servo
- removed link wrist_pan_servo_bracket_f3
- added link head_cam_depth_frame, mass 0.000001
- added link head_cam_depth_optical_frame, mass 0.000001
- added link head_cam_link, mass 1.0; collision mesh filename=package://robbie_description/meshes/kinect.stl scale=0.001 0.001 0.001; visual mesh filename=package://robbie_description/meshes/kinect.stl scale=0.001 0.001 0.001
- added link head_cam_rgb_frame, mass 0.000001
- added link head_cam_rgb_optical_frame, mass 0.000001
- added link kinect_rgb_frame, mass 0.000001
- added link lower_torso; visual mesh filename=package://robbie_description/meshes/chest_lower.stl scale=0.001 0.001 0.001
- added link right_wrist_yaw_bracket_f2, mass 0.02; collision mesh filename=package://robbie_description/meshes/F2.stl scale=0.001 0.001 0.001; visual mesh filename=package://robbie_description/meshes/F2.stl scale=0.001 0.001 0.001
- added link wrist_yaw_servo, mass 0.055; collision mesh filename=package://robbie_description/meshes/ax12_box2.stl scale=0.001 0.001 0.001; visual mesh filename=package://robbie_description/meshes/ax12_box2.stl scale=0.001 0.001 0.001
- added link wrist_yaw_servo_bracket_f3, mass 0.01; collision mesh filename=package://robbie_description/meshes/F3.stl scale=0.001 0.001 0.001; visual mesh filename=package://robbie_description/meshes/F3.stl scale=0.001 0.001 0.001
- link base_link: geometry collision box size=0.41 0.35 0.065; visual box size=0.41 0.35 0.065
- link deck_link: mass 0.2 -> None; geometry visual mesh filename=package://robbie_description/meshes/drive_base.stl scale=0.001 0.001 0.001
- link gripper_bracket_f2: geometry collision mesh filename=package://robbie_description/meshes/F2.stl scale=0.001 0.001 0.001; visual mesh filename=package://robbie_description/meshes/F2.stl scale=0.001 0.001 0.001
- link gripper_bracket_f3: geometry collision mesh filename=package://robbie_description/meshes/F3.stl scale=0.001 0.001 0.001; visual mesh filename=package://robbie_description/meshes/F3.stl scale=0.001 0.001 0.001
- link gripper_servo: geometry collision mesh filename=package://robbie_description/meshes/ax12_box2.stl scale=0.001 0.001 0.001; visual mesh filename=package://robbie_description/meshes/ax12_box2.stl scale=0.001 0.001 0.001
- link head_link: geometry visual mesh filename=package://robbie_description/meshes/head1.stl scale=0.001 0.001 0.001
- link head_pan_bracket: geometry collision mesh filename=package://robbie_description/meshes/F3.stl scale=0.001 0.001 0.001; visual mesh filename=package://robbie_description/meshes/F3.stl scale=0.001 0.001 0.001
- link head_pan_link: geometry collision mesh filename=package://robbie_description/meshes/ax12_box2.stl scale=0.001 0.001 0.001; visual mesh filename=package://robbie_description/meshes/ax12_box2.stl scale=0.001 0.001 0.001
- link head_tilt_bracket: geometry collision mesh filename=package://robbie_description/meshes/F2.stl scale=0.001 0.001 0.001; visual mesh filename=package://robbie_description/meshes/F2.stl scale=0.001 0.001 0.001
- link head_tilt_link: geometry collision mesh filename=package://robbie_description/meshes/ax12_box2.stl scale=0.001 0.001 0.001; visual mesh filename=package://robbie_description/meshes/ax12_box2.stl scale=0.001 0.001 0.001
- link kinect_depth_frame: mass 0.0001 -> 0.000001
- link kinect_depth_optical_frame: mass 0.0001 -> 0.000001
- link kinect_rgb_optical_frame: mass 0.001 -> 0.000001
- link left_gripper_bracket_f2: geometry collision mesh filename=package://robbie_description/meshes/F2.stl scale=0.001 0.001 0.001; visual mesh filename=package://robbie_description/meshes/F2.stl scale=0.001 0.001 0.001
- link left_gripper_bracket_f3: geometry collision mesh filename=package://robbie_description/meshes/F3.stl scale=0.001 0.001 0.001; visual mesh filename=package://robbie_description/meshes/F3.stl scale=0.001 0.001 0.001
- link left_gripper_servo: geometry collision mesh filename=package://robbie_description/meshes/ax12_box2.stl scale=0.001 0.001 0.001; visual mesh filename=package://robbie_description/meshes/ax12_box2.stl scale=0.001 0.001 0.001
- link left_wrist_pan_servo_bracket_f3: geometry collision mesh filename=package://robbie_description/meshes/F3.stl scale=0.001 0.001 0.001; visual mesh filename=package://robbie_description/meshes/F3.stl scale=0.001 0.001 0.001
- link left_wrist_tilt_bracket_f2: geometry collision mesh filename=package://robbie_description/meshes/F2.stl scale=0.001 0.001 0.001; visual mesh filename=package://robbie_description/meshes/F2.stl scale=0.001 0.001 0.001
- link left_wrist_tilt_servo: geometry collision mesh filename=package://robbie_description/meshes/ax12_box2.stl scale=0.001 0.001 0.001; visual mesh filename=package://robbie_description/meshes/ax12_box2.stl scale=0.001 0.001 0.001
- link left_wrist_yaw_bracket_f2: geometry collision mesh filename=package://robbie_description/meshes/F2.stl scale=0.001 0.001 0.001; visual mesh filename=package://robbie_description/meshes/F2.stl scale=0.001 0.001 0.001
- link left_wrist_yaw_servo: geometry collision mesh filename=package://robbie_description/meshes/ax12_box2.stl scale=0.001 0.001 0.001; visual mesh filename=package://robbie_description/meshes/ax12_box2.stl scale=0.001 0.001 0.001
- link neck_link: geometry collision mesh filename=package://robbie_description/meshes/F3.stl scale=0.001 0.001 0.001; visual mesh filename=package://robbie_description/meshes/F3.stl scale=0.001 0.001 0.001
- link pan_link: geometry collision cylinder length=0.005 radius=0.1; visual cylinder length=0.005 radius=0.1
- link wrist_tilt_bracket_f2: geometry collision mesh filename=package://robbie_description/meshes/F2.stl scale=0.001 0.001 0.001; visual mesh filename=package://robbie_description/meshes/F2.stl scale=0.001 0.001 0.001
- link wrist_tilt_servo: geometry collision mesh filename=package://robbie_description/meshes/ax12_box2.stl scale=0.001 0.001 0.001; visual mesh filename=package://robbie_description/meshes/ax12_box2.stl scale=0.001 0.001 0.001
Joints:
- removed joint camera_link
- removed joint left_arm_wrist_pan_bracket
- removed joint left_arm_wrist_pan_joint
- removed joint left_wheel_joint
- removed joint right_arm_wrist_pan_bracket
- removed joint right_arm_wrist_pan_joint
- removed joint right_arm_wrist_tilt_bracket
- removed joint right_wheel_joint
- added joint base_l_wheel_joint: type fixed, parent base_link, child left_wheel, origin xyz=0.1 -0.2 -0.04 rpy=0 0 0
- added joint base_r_wheel_joint: type fixed, parent base_link, child right_wheel, origin xyz=0.1 0.2 -0.04 rpy=0 0 0
- added joint head_cam_depth_joint: type fixed, parent head_cam_link, child head_cam_depth_frame, origin xyz=0 0.0125 0.015 rpy=0 0 0
- added joint head_cam_depth_optical_joint: type fixed, parent head_cam_depth_frame, child head_cam_depth_optical_frame, origin xyz=0 0 0 rpy=-1.57075 0 -1.57075
- added joint head_cam_joint: type fixed, parent head_link, child head_cam_link, origin xyz=0.15 0.11 0.13 rpy=0 0.1 0
- added joint head_cam_rgb_joint: type fixed, parent head_cam_link, child head_cam_rgb_frame, origin xyz=0 -0.0125 0.015 rpy=0 0 0
- added joint head_cam_rgb_optical_joint: type fixed, parent head_cam_rgb_frame, child head_cam_rgb_optical_frame, origin xyz=0 0 0 rpy=-1.57075 0 -1.57075
- added joint kinect_rgb_joint: type fixed, parent kinect_link, child kinect_rgb_frame, origin xyz=0 -0.0125 0.015 rpy=0 0 0
- added joint left_arm_wrist_yaw_attach: type fixed, parent left_forearm_link, child left_wrist_pan_servo_bracket_f3, origin xyz=0. 0 0 rpy=0 0 0
- added joint right_arm_wrist_tilt1_bracket: type fixed, parent right_wrist_yaw_bracket_f2, child wrist_tilt_bracket_f2, origin xyz=0.053 0 0.0 rpy=0 0 0, axis 0 0 1
- added joint right_arm_wrist_tilt_joint: type revolute, parent wrist_tilt_bracket_f2, child wrist_tilt_servo, origin xyz=0 0 0 rpy=0 0 0, axis 0 1 0, limit lower=-1.57 upper=1.57 effort=10 velocity=1
- added joint right_arm_wrist_yaw_bracket: type fixed, parent right_forearm_link, child wrist_yaw_servo_bracket_f3, origin xyz=0.0 0.0 0.0 rpy=0 0 0
- added joint right_arm_wrist_yaw_bracket1: type fixed, parent wrist_yaw_servo_bracket_f3, child wrist_yaw_servo, origin xyz=0.04 0 0.0 rpy=0 0 0, axis 0 0 1, limit lower=-2.61 upper=2.61 effort=10 velocity=1
- added joint torso_lower_link: type fixed, parent pan_link, child lower_torso, origin xyz=0.0 0.005 0. rpy=0 0 0
- joint base_footprint_joint: origin xyz=-0.1 0 0 rpy=0 0 0 -> xyz=-0.1 0 0.15 rpy=0 0 0
- joint base_link_joint: origin xyz=-0.1 0 .36 rpy=0 0 0 -> xyz=0 0 0.138 rpy=0 0 0
- joint castor_wheel_joint_l: origin xyz=-0.20 -0.13 0.05 rpy=0 0 0 -> xyz=-0.20 -0.13 -0.1 rpy=0 0 0
- joint castor_wheel_joint_r: origin xyz=-0.20 0.13 0.05 rpy=0 0 0 -> xyz=-0.20 0.13 -0.1 rpy=0 0 0
- joint chest_link: origin xyz=0.02 0 0.03 rpy=0 0 0 -> xyz=0.065 0 -0.04 rpy=0 0 0
- joint head_joint: origin xyz=-0.02 -0.097 -0.45 rpy=0 0 0 -> xyz=-0.02 -0.097 0 rpy=0 0 0
- joint head_pan_joint: limit lower=-2 upper=2 effort=10 velocity=0 -> lower=-2 upper=2 effort=10 velocity=1
- joint head_tilt_joint: limit lower=-2.6 upper=2.6 effort=10 velocity=0 -> lower=-2.6 upper=2.6 effort=10 velocity=1
- joint head_tilt_mod_joint: limit lower=-2.6 upper=2.6 effort=10 velocity=0 -> lower=-2.6 upper=2.6 effort=10 velocity=1
- joint head_tilt_servo: origin xyz=-0.05 0. 0.15 rpy=0 0 0 -> xyz=-0.0 0. 0.05 rpy=0 0 0
- joint kinect_depth_joint: origin xyz=0 0.018 0 rpy=0 0 0 -> xyz=0 0.0125 0.015 rpy=0 0 0
- joint kinect_depth_optical_joint: origin xyz=0 0 0 rpy=-1.570795 0 -1.570795 -> xyz=0 0 0 rpy=-1.57075 0 -1.57075; parent kinect_link -> kinect_depth_frame
- joint kinect_joint: origin xyz=0.2 0 0.26 rpy=0 0 0 -> xyz=0.2 0 0.32 rpy=0 0 0
- joint kinect_rgb_optical_joint: origin xyz=0 0 0 rpy=-1.570795 0 -1.570795 -> xyz=0 0 0 rpy=-1.57075 0 -1.57075; parent kinect_depth_optical_frame -> kinect_rgb_frame
- joint left_arm_elbow_joint: limit lower=-2.20 upper=0.17 effort=10 velocity=0 -> lower=-2.20 upper=0.17 effort=10 velocity=1; origin xyz=0.01 0.01 0.0 rpy=0 -1.57 0 -> xyz=0 0 0 rpy=0 -0 0
- joint left_arm_finger_link_l: origin xyz=0. 0.03 -0.04 rpy=0 0 0 -> xyz=0.08 0.04 0 rpy=0 0 0
- joint left_arm_finger_link_r: origin xyz=0 0.03 0.03 rpy=0 0 0 -> xyz=0.08 -0.03 0 rpy=0 0 0
- joint left_arm_forearm_link: origin xyz=-0.08 -0.0 -0.0 rpy=1.57 0 0 -> xyz=0.31 -0.0 -0.0 rpy=0 0 0
- joint left_arm_gripper_bracket: origin xyz=0.0 0.035 0.0 rpy=0 1.57 0 -> xyz=0.04 0 0.0 rpy=3.14 0 0
- joint left_arm_gripper_joint: axis 1 0 0 -> 0 0 1; limit lower=-1.0 upper=0.3 effort=10 velocity=0 -> lower=-1.0 upper=0.3 effort=10 velocity=1
- joint left_arm_gripper_servo: origin xyz=0.0 0.02 -0.02 rpy=0 3.14 0 -> xyz=0.02 -0.02 -0. rpy=0 0 0
- joint left_arm_lift_joint: limit lower=-1.57 upper=1.57 effort=10 velocity=0 -> lower=-1.57 upper=1.57 effort=10 velocity=1; origin xyz=0 0.02 -0.04 rpy=0 -1.57 0 -> xyz=0 0.08 -0.04 rpy=0 0 0
- joint left_arm_rotate_joint: axis 0 0 -1 -> 1 0 0; limit lower=0.2 upper=3.14 effort=10 velocity=0 -> lower=-2.6 upper=2.6 effort=10 velocity=1; origin xyz=0 0.06 -0.055 rpy=0 0 0 -> xyz=0.24 0 0 rpy=0 0 0
- joint left_arm_tilt_joint: limit lower=-1.34 upper=0.1 effort=10 velocity=0 -> lower=-1.34 upper=0.03 effort=10 velocity=1; origin xyz=-0.045 0.145 0.105 rpy=0 0 0 -> xyz=0.003 0.142 -0.05 rpy=0 0 0
- joint left_arm_wrist_tilt_joint: axis 1 0 0 -> 0 1 0; limit lower=-1.57 upper=1.57 effort=10 velocity=0 -> lower=-1.57 upper=1.57 effort=10 velocity=1
- joint left_arm_wrist_yaw_bracket: limit lower=-1.57 upper=1.57 effort=10 velocity=0 -> lower=-1.57 upper=1.57 effort=10 velocity=1; origin xyz=-0.0 0.052 0.0 rpy=0 0 0 -> xyz=0.055 0 0.0 rpy=0 0 0
- joint left_arm_wrist_yaw_joint: axis 0 0 -1 -> 0 0 1; limit lower=-1.57 upper=1.57 effort=10 velocity=0 -> lower=-1.57 upper=1.57 effort=10 velocity=1; origin xyz=-0.04 0.05 0 rpy=0 0 0 -> xyz=0.0 0 0 rpy=0 0 0
- joint left_elbow_link: origin xyz=0.01 0 -0.17 rpy=0 0 0 -> xyz=-0.01 0 0.008 rpy=0 0 0
- joint left_gripper_joint: origin xyz=0 0.06 -0.01 rpy=1.570795 0 1.570795 -> xyz=0.06 -0.01 0 rpy=0 0 0
- joint pan_joint: origin xyz=0.1 0 0.275 rpy=0 0 0 -> xyz=0 0 0.35 rpy=0 0 0
- joint right_arm_elbow_joint: limit lower=-2.20 upper=0.1 effort=10 velocity=0 -> lower=-2.20 upper=0.1 effort=10 velocity=10; origin xyz=0.01 0.01 0.0 rpy=0 -1.57 0 -> xyz=0.01 0.01 0.0 rpy=0 0 0
- joint right_arm_finger_link_l: origin xyz=0.03 0.04 0.0 rpy=0 1.57 -1.57 -> xyz=0.08 0.04 0 rpy=0 0 0
- joint right_arm_finger_link_r: origin xyz=0 0.03 0.03 rpy=0 0 0 -> xyz=0.08 -0.03 0 rpy=0 0 0
- joint right_arm_forearm_link: origin xyz=-0.08 -0.0 -0.0 rpy=1.57 0 0 -> xyz=0.31 -0.0 -0.0 rpy=0 0 0
- joint right_arm_gripper_bracket: origin xyz=0.025 0.025 0.0 rpy=1.57 1.57 0 -> xyz=0.04 0 0.0 rpy=0 0 0; parent wrist_tilt_bracket_f2 -> wrist_tilt_servo
- joint right_arm_gripper_joint: axis 1 0 0 -> 0 0 1; limit lower=-0.36 upper=0.28 effort=10 velocity=0 -> lower=-0.1 upper=0.50 effort=10 velocity=1; origin xyz=0 0.0 0.0 rpy=0 1.57 -1.57 -> xyz=0 0.0 0.0 rpy=0 0 0
- joint right_arm_gripper_servo: origin xyz=0.0 0.02 0.02 rpy=-1.57 0 1.57 -> xyz=0.02 -0.015 0.0 rpy=0 0 0
- joint right_arm_lift_joint: limit lower=-1.57 upper=1.57 effort=10 velocity=0 -> lower=-1.57 upper=1.57 effort=10 velocity=1; origin xyz=-0.0 -0.077 -0.04 rpy=0 -1.57 0 -> xyz=0 -0.078 -0.042 rpy=0 0 0
- joint right_arm_rotate_joint: axis 0 0 -1 -> 1 0 0; limit lower=-3.14 upper=0.2 effort=10 velocity=0 -> lower=-2.6 upper=2.6 effort=10 velocity=1; origin xyz=0 0 -0.065 rpy=0 0 0 -> xyz=0.255 -0.01 0 rpy=0 0 0
- joint right_arm_tilt_joint: limit lower=-1.34 upper=0.1 effort=10 velocity=0 -> lower=-1.34 upper=0.1 effort=10 velocity=1; origin xyz=-0.045 -0.145 0.105 rpy=0 0 0 -> xyz=0 -0.14 -0.045 rpy=0 0 0
- joint right_arm_wrist_yaw_joint: axis 0 1 0 -> 0 0 1; child wrist_tilt_bracket_f2 -> right_wrist_yaw_bracket_f2; limit lower=-1.57 upper=1.57 effort=10 velocity=0 -> lower=-2.61 upper=2.61 effort=10 velocity=1; origin xyz=-0.04 0.05 0 rpy=-1.57 0 1.57 -> xyz=0.0 0 0.0 rpy=0 0 0; parent wrist_tilt_servo -> wrist_yaw_servo
- joint right_elbow_link: origin xyz=0.01 0 -0.17 rpy=0 0 0 -> xyz=-0.01 0 0.01 rpy=0 0 0
- joint right_gripper_joint: origin xyz=0 0.06 0.01 rpy=-1.570795 0 1.570795 -> xyz=0.06 -0.01 0 rpy=0 0 0
- joint torso_link: origin xyz=0.05 0 0.26 rpy=0 0 0 -> xyz=0.0 0.005 0.465 rpy=0 0 0
