Commit message: add robbie_gazebo and control

File: robbie_description/urdf/rob_inmoov.xacro (robot description, xacro)
@@ -11,5 +11,5 @@
     <property name="MESH_EXT" value="stl"/>
     <xacro:include filename="$(find robbie_description)/urdf/robbie_hardware.xacro" />
-<xacro:my_box name="base_link" lwh="0.41 0.35 0.064" xyz="0 0 -0.032" rpy="0 0 0" mass="0.1" material="Gazebo/FlatBlack">
+<xacro:my_box name="base_link" lwh="0.41 0.35 0.065" xyz="0 0 -0.032" rpy="0 0 0" mass="0.1" material="Gazebo/FlatBlack">
 	        <xacro:gold />
         </xacro:my_box>
@@ -35,11 +35,29 @@
 		<xacro:grey1 />
 	</xacro:my_cylinder>
-  <xacro:my_cylinder name="deck_link" l="0.520" r="0.175" xyz="0 0 -0.26" rpy="0 0 0" mass="0.2" material="Gazebo/grey">
+  <!--<xacro:my_cylinder name="deck_link" l="0.520" r="0.175" xyz="0 0 -0.26" rpy="0 0 0" mass="0.2" material="Gazebo/grey">
 			<xacro:black />
-		</xacro:my_cylinder>
- <xacro:my_cylinder name="pan_link" l="0.02" r="0.17" xyz="0 0 0" rpy="0 0 0" mass="0.2" material="Gazebo/grey">
-			<xacro:blue1 />
+		</xacro:my_cylinder>-->
+  <link name="deck_link" >
+   <visual>
+      <geometry>
+        <mesh filename="package://robbie_description/meshes/drive_base.stl" scale="${M_SCALE} ${M_SCALE} ${M_SCALE}"/>
+      </geometry>
+         <xacro:yellow2/>
+      <origin rpy="0 0 1.57" xyz=" 0.015 -0.175 -0"/>
+    </visual>
+  </link>
+ <xacro:my_cylinder name="pan_link" l="0.005" r="0.1" xyz="0.0 0 -0.02" rpy="0 0 0" mass="0.2" material="Gazebo/grey">
+			<xacro:yellow2 />
 		</xacro:my_cylinder>
 <!-- ##############################   upper torso   ##################333333-->
+<link name="lower_torso" >
+   <visual>
+      <geometry>
+        <mesh filename="package://robbie_description/meshes/chest_lower.stl" scale="${M_SCALE} ${M_SCALE} ${M_SCALE}"/>
+      </geometry>
+         <xacro:yellow2/>
+      <origin rpy="0 0 1.57" xyz="0 0 0"/>
+    </visual>
+  </link>
 <link name="upper_torso" >
    <visual>
@@ -146,5 +164,5 @@
         <mesh filename="package://robbie_description/meshes/left_shoulder_assy.stl" scale="${M_SCALE} ${M_SCALE} ${M_SCALE}"/>
       </geometry>
-       <xacro:grey1 />
+       <xacro:black />
       <origin rpy="-1.57 0 1.57" xyz="0 -0.06 0"/>
     </visual>
@@ -280,7 +298,7 @@
       </collision>
     </link>
-    <xacro:my_cylinder name="camera_link" l="0.035" r="0.01" xyz="0 0 0" rpy="0 1.57 0" mass="0.1" material="Gazebo/Grey">
+    <!--<xacro:my_cylinder name="camera_link" l="0.035" r="0.01" xyz="0 0 0" rpy="0 1.57 0" mass="0.1" material="Gazebo/Grey">
       <xacro:grey1 />
-	</xacro:my_cylinder>
+	</xacro:my_cylinder>-->
 <!-- virtal joints-->
 <link name="right_gripper_link">
@@ -316,17 +334,17 @@
     	<parent link="base_footprint" />
     	<child link="base_link" />
-    	<origin xyz="-0.1 0 0.08" rpy="0 0 0" />
+    	<origin xyz="-0.1 0 0.15" rpy="0 0 0" />
 	</joint>
 <joint name="base_link_joint" type="fixed">
     	<parent link="base_link" />
     	<child link="deck_link" />
-    	<origin xyz="0 0 0.51" rpy="0 0 0" />
-	</joint>
-  <joint name="left_wheel_joint" type="fixed">
+    	<origin xyz="0 0 0.138" rpy="0 0 0" />
+	</joint>
+  <joint name="base_l_wheel_joint" type="fixed">
     	<parent link="base_link" />
     	<child link="left_wheel" />
     	<origin xyz="0.1 -0.2 -0.04" rpy="0 0 0" />
 	</joint>
-  <joint name="right_wheel_joint" type="fixed">
+  <joint name="base_r_wheel_joint" type="fixed">
     	<parent link="base_link" />
     	<child link="right_wheel" />
@@ -347,12 +365,17 @@
     	<parent link="deck_link" />
     	<child link="pan_link" />
-    	<origin xyz="0.0 0 0" rpy="0 0 0" />
+    	<origin xyz="0 0 0.35" rpy="0 0 0" />
         <axis xyz="0 0 1" />
         <limit lower="-1" upper="1" effort="10" velocity="0" />
+	</joint>
+  <joint name="torso_lower_link" type="fixed">
+    	<parent link="pan_link" />
+    	<child link="lower_torso" />
+    	<origin xyz="0.0 0.005 0." rpy="0 0 0" />
 	</joint>
   <joint name="torso_link" type="fixed">
     	<parent link="pan_link" />
     	<child link="upper_torso" />
-    	<origin xyz="0.0 0 0.47" rpy="0 0 0" />
+    	<origin xyz="0.0 0.005 0.465" rpy="0 0 0" />
 	</joint>
 <joint name="chest_link" type="fixed">
@@ -366,5 +389,5 @@
     	<origin xyz="0 -0.14 -0.045" rpy="0 0 0" />
         <axis xyz="1 0 0" />
-        <limit lower="-1.34" upper="0.1" effort="10" velocity="0" />
+        <limit lower="-1.34" upper="0.1" effort="10" velocity="1" />
 	</joint>
 <joint name="right_arm_lift_joint" type="revolute">
@@ -373,12 +396,12 @@
     	<origin xyz="0 -0.078 -0.042" rpy="0 0 0" />
         <axis xyz="0 1 0" />
-        <limit lower="-1.57" upper="1.57" effort="10" velocity="0" />
+        <limit lower="-1.57" upper="1.57" effort="10" velocity="1" />
 	</joint>
 <joint name="right_arm_rotate_joint" type="revolute">
     	<parent link="right_shoulder_lift" />
     	<child link="right_shoulder_rotate" />
-    	<origin xyz="0.255 0 0" rpy="0 0 0" />
+    	<origin xyz="0.255 -0.01 0" rpy="0 0 0" />
         <axis xyz="1 0 0" />
-        <limit lower="-3.14" upper="0.2" effort="10" velocity="0" />
+        <limit lower="-2.6" upper="2.6" effort="10" velocity="1" />
 	</joint>
 <joint name="right_elbow_link" type="fixed">
@@ -392,5 +415,5 @@
     <origin xyz="0.01 0.01 0.0" rpy="0 0 0" />
     <axis xyz="0 1 0" />
-   <limit lower="-2.20" upper="0.1" effort="10" velocity="0" />
+   <limit lower="-2.20" upper="0.1" effort="10" velocity="10" />
   </joint>
   <joint name="right_arm_forearm_link" type="fixed">
@@ -410,5 +433,5 @@
     	<origin xyz="0.04 0 0.0" rpy="0 0 0" />
         <axis xyz="0 0 1" />
-    	<limit lower="-2.61" upper="2.61" effort="10" velocity="0" />
+    	<limit lower="-2.61" upper="2.61" effort="10" velocity="1" />
       	<dynamics damping="0.0"/>
 	</joint>
@@ -418,5 +441,5 @@
     	<origin xyz="0.0 0 0.0" rpy="0 0 0" />
         <axis xyz="0 0 1" />
-    	<limit lower="-2.61" upper="2.61" effort="10" velocity="0" />
+    	<limit lower="-2.61" upper="2.61" effort="10" velocity="1" />
 	</joint>
 <joint name="right_arm_wrist_tilt1_bracket" type="fixed">
@@ -432,5 +455,5 @@
     	<origin xyz="0 0 0" rpy="0 0 0" />
         <axis xyz="0 1 0" />
-    	<limit lower="-1.57" upper="1.57" effort="10" velocity="0" />
+    	<limit lower="-1.57" upper="1.57" effort="10" velocity="1" />
       	<dynamics damping="0.0"/>
 	</joint>
@@ -456,5 +479,5 @@
     	<origin xyz="0 0.0 0.0" rpy="0 0 0" />
         <axis xyz="0 0 1" />
-    	<limit lower="-0.1" upper="0.50" effort="10" velocity="0" />
+    	<limit lower="-0.1" upper="0.50" effort="10" velocity="1" />
       	<dynamics damping="0.0"/>
 	</joint>
@@ -476,5 +499,5 @@
     	<origin xyz="0.003 0.142 -0.05" rpy="0 0 0" />
         <axis xyz="-1 0 0" />
-        <limit lower="-1.34" upper="0.1" effort="10" velocity="0" />
+        <limit lower="-1.34" upper="0.03" effort="10" velocity="1" />
 	</joint>
 <joint name="left_arm_lift_joint" type="revolute">
@@ -483,5 +506,5 @@
     	<origin xyz="0 0.08 -0.04" rpy="0 0 0" />
         <axis xyz="0 1 0" />
-        <limit lower="-1.57" upper="1.57" effort="10" velocity="0" />
+        <limit lower="-1.57" upper="1.57" effort="10" velocity="1" />
 	</joint>
 <joint name="left_arm_rotate_joint" type="revolute">
@@ -490,5 +513,5 @@
     	<origin xyz="0.24 0 0" rpy="0 0 0" />
         <axis xyz="1 0 0" />
-        <limit lower="-0.2" upper="3.14" effort="10" velocity="0" />
+        <limit lower="-2.6" upper="2.6" effort="10" velocity="1" />
 	</joint>
 <joint name="left_elbow_link" type="fixed">
@@ -502,5 +525,5 @@
     <origin xyz="0 0 0" rpy="0 -0 0" />
     <axis xyz="0 1 0" />
-   <limit lower="-2.20" upper="0.17" effort="10" velocity="0" />
+   <limit lower="-2.20" upper="0.17" effort="10" velocity="1" />
   </joint>
  <joint name="left_arm_forearm_link" type="fixed">
@@ -527,5 +550,5 @@
     	<origin xyz="0.0 0 0" rpy="0 0 0" />
         <axis xyz="0 0 1" />
-    	<limit lower="-1.57" upper="1.57" effort="10" velocity="0" />
+    	<limit lower="-1.57" upper="1.57" effort="10" velocity="1" />
       	<dynamics damping="0.0"/>
 	</joint>
@@ -535,5 +558,5 @@
     	<origin xyz="0.055 0 0.0" rpy="0 0 0" />
         <axis xyz="1 0 0" />
-    	<limit lower="-1.57" upper="1.57" effort="10" velocity="0" />
+    	<limit lower="-1.57" upper="1.57" effort="10" velocity="1" />
       	<dynamics damping="0.0"/>
         </joint>
@@ -544,5 +567,5 @@
     	<origin xyz="-0 -0.0 0" rpy="0 0 0" />
         <axis xyz="0 1 0" />
-    	<limit lower="-1.57" upper="1.57" effort="10" velocity="0" />
+    	<limit lower="-1.57" upper="1.57" effort="10" velocity="1" />
       	<dynamics damping="0.0"/>
 	</joint>
@@ -550,5 +573,5 @@
     	<parent link="left_wrist_tilt_servo" />
     	<child link="left_gripper_bracket_f3" />
-    	<origin xyz="0.04 0 0.0" rpy="0 0 0" />
+    	<origin xyz="0.04 0 0.0" rpy="3.14 0 0" />
 	</joint>
    <joint name="left_arm_gripper_servo" type="fixed">
@@ -568,5 +591,5 @@
     	<origin xyz="0 0.0 0.0" rpy="0 0 0" />
         <axis xyz="0 0 1" />
-    	<limit lower="-1.0" upper="0.3" effort="10" velocity="0" />
+    	<limit lower="-1.0" upper="0.3" effort="10" velocity="1" />
       	<dynamics damping="0.0"/>
 	</joint>
@@ -593,5 +616,5 @@
     	<origin xyz="0 0 0.0" rpy="0 0 0" />
     	<axis xyz="0 1 0" />
-    	<limit lower="-2.6" upper="2.6" effort="10" velocity="0" />
+    	<limit lower="-2.6" upper="2.6" effort="10" velocity="1" />
       	<dynamics damping="0.0"/>
 	</joint>
@@ -602,5 +625,5 @@
     	<origin xyz="0 0 0.0" rpy="0 0 0" />
     	<axis xyz="0 1 0" />
-    	<limit lower="-2.6" upper="2.6" effort="10" velocity="0" />
+    	<limit lower="-2.6" upper="2.6" effort="10" velocity="1" />
       	<dynamics damping="0.0"/>
 	</joint>
@@ -617,5 +640,5 @@
         <origin xyz="0 0 0.0" rpy="0 0 0" />
     	<axis xyz="0 0 1" />
-    	<limit lower="-2" upper="2" effort="10" velocity="0" />
+    	<limit lower="-2" upper="2" effort="10" velocity="1" />
       	<dynamics damping="0.0"/>
 	</joint>
@@ -635,13 +658,13 @@
     	<origin xyz="-0.02 -0.097 0" rpy="0 0 0" />
 	</joint>
-   <joint name="camera_link" type="fixed">
+   <!--<joint name="camera_link" type="fixed">
     	<parent link="head_link" />
     	<child link="camera_link" />
     	<origin xyz="0.13 0.1 0.6" rpy="0 0 0" />
-	</joint>
+	</joint>-->
   <joint name="kinect_joint" type="fixed">
     	<parent link="base_link" />
     	<child link="kinect_link" />
-    	<origin xyz="0.2 0 0.33" rpy="0 0 0" />
+    	<origin xyz="0.2 0 0.32" rpy="0 0 0" />
 	</joint>
 <joint name="kinect_depth_joint" type="fixed">
@@ -704,5 +727,5 @@
     	<parent link="head_link" />
     	<child link="head_cam_link" />
-    	<origin xyz="0.15 0.11 0.13" rpy="0 0 0" />
+    	<origin xyz="0.15 0.11 0.13" rpy="0 0.1 0" />
 	</joint>
 <joint name="head_cam_depth_joint" type="fixed">

File: robbie_description/urdf/robbie_hardware.xacro (robot description, xacro)
@@ -1,4 +1,4 @@
 <?xml version="1.0"?>
-<robot name="hector_base" xmlns:xacro="http://ros.org/wiki/xacro">
+<robot name="robbie" xmlns:xacro="http://ros.org/wiki/xacro">
   <!-- ============================  A Few Color Macros  ============================ -->
 	<xacro:macro name="black">
@@ -7,6 +7,6 @@
 		</material>
 	</xacro:macro>
-	<xacro:macro name="white">
-		<material name="white">
+	<xacro:macro name="White">
+		<material name="White">
 			<color rgba="1.0 1.0 1.0 1.0"/>
 		</material>
@@ -120,5 +120,5 @@
              <xacro:default_inertial mass="0.02" />
         </link>
-        <xacro:default_gazebo name="${name}" material="Gazebo/WhiteEmissive" />
+        <xacro:default_gazebo name="${name}" material="Gazebo/White" />
 	</xacro:macro>
 	<xacro:macro name="F3_bracket" params="name xyz rpy">
@@ -141,5 +141,5 @@
              <xacro:default_inertial mass="0.01" />
         </link>
-        <xacro:default_gazebo name="${name}" material="Gazebo/WhiteEmissive" />
+        <xacro:default_gazebo name="${name}" material="Gazebo/White" />
 	</xacro:macro>
 	<xacro:macro name="bracket_f3" params="name xyz rpy">
@@ -160,5 +160,5 @@
              <xacro:default_inertial mass="0.02" />
         </link>
-        <xacro:default_gazebo name="${name}" material="Gazebo/WhiteEmissive" />
+        <xacro:default_gazebo name="${name}" material="Gazebo/White" />
 	</xacro:macro>
 	<xacro:macro name="bracket2" params="name xyz rpy">
@@ -179,5 +179,5 @@
              <xacro:default_inertial mass="0.01" />
         </link>
-        <xacro:default_gazebo name="${name}" material="Gazebo/WhiteEmissive" />
+        <xacro:default_gazebo name="${name}" material="Gazebo/White" />
 	</xacro:macro>
         <xacro:macro name="bracket3" params="name xyz rpy">
@@ -198,24 +198,5 @@
              <xacro:default_inertial mass="0.01" />
         </link>
-        <xacro:default_gazebo name="${name}" material="Gazebo/WhiteEmissive" />
-	</xacro:macro>
-        <xacro:macro name="h_beam" params="name xyz rpy">
-		<link name="${name}">
-			<visual>
-				<origin xyz="${xyz}" rpy="${rpy}" />
-				<geometry>
-					<box size="0.025 0.11 0.01" />
-				</geometry>
-				<xacro:bracket_color />
-             </visual>
-             <collision>
-				<origin xyz="${xyz}" rpy="${rpy}" />
-					<geometry>
-					<box size="0.025 0.11 0.01" />
-					</geometry>
-             </collision>
-             <xacro:default_inertial mass="0.01" />
-        </link>
-        <xacro:default_gazebo name="${name}" material="Gazebo/WhiteEmissive" />
+        <xacro:default_gazebo name="${name}" material="Gazebo/White" />
 	</xacro:macro>
         <xacro:macro name="my_box" params="name lwh xyz rpy mass material *rviz_color">
@@ -233,4 +214,5 @@
 						<box size="${lwh}" />
 					</geometry>
+              <xacro:default_inertial mass="0.01" />
              </collision>
         </link>
@@ -259,7 +241,7 @@
 		<inertial>
 			<mass value="${mass}" />
-			<inertia ixx="0.001" ixy="0.0" ixz="0.0"
-                     iyy="0.001" iyz="0.0"
-                     izz="0.001" />
+			<inertia ixx="0.0001" ixy="0.0" ixz="0.0"
+                     iyy="0.0001" iyz="0.0"
+                     izz="0.0001" />
 			</inertial>
     </xacro:macro>
@@ -268,5 +250,5 @@
 			<material>${material}</material>
 			<selfCollide>false</selfCollide>
-			<turnGravityOff>true</turnGravityOff>
+			<turnGravityOff>false</turnGravityOff>
 		</gazebo>
     </xacro:macro>

Commit message: pre reconfigure

File: robbie_description/urdf/rob_inmoov.urdf (robot description, URDF)
Before this commit: robot robbie, 63 links, 62 joints
Links:
- removed link head_cam_depth_frame
- removed link head_cam_depth_optical_frame
- removed link head_cam_link
- removed link head_cam_rgb_frame
- removed link head_cam_rgb_optical_frame
- added link camera_depth_frame, mass 0.000001
- added link camera_depth_optical_frame, mass 0.000001
- added link camera_link, mass 1.0; collision mesh filename=package://robbie_description/meshes/kinect.stl scale=0.001 0.001 0.001; visual mesh filename=package://robbie_description/meshes/kinect.stl scale=0.001 0.001 0.001
- added link camera_rgb_frame, mass 0.000001
- added link camera_rgb_optical_frame, mass 0.000001
Joints:
- removed joint head_cam_depth_joint
- removed joint head_cam_depth_optical_joint
- removed joint head_cam_joint
- removed joint head_cam_rgb_joint
- removed joint head_cam_rgb_optical_joint
- added joint camera_depth_joint: type fixed, parent camera_link, child camera_depth_frame, origin xyz=0 0.0125 0.015 rpy=0 0 0
- added joint camera_depth_optical_joint: type fixed, parent camera_depth_frame, child camera_depth_optical_frame, origin xyz=0 0 0 rpy=-1.57075 0 -1.57075
- added joint camera_joint: type fixed, parent head_link, child camera_link, origin xyz=0.15 0.11 0.13 rpy=0 0.1 0
- added joint camera_rgb_joint: type fixed, parent camera_link, child camera_rgb_frame, origin xyz=0 -0.0125 0.015 rpy=0 0 0
- added joint camera_rgb_optical_joint: type fixed, parent camera_rgb_frame, child camera_rgb_optical_frame, origin xyz=0 0 0 rpy=-1.57075 0 -1.57075

File: robbie_description/urdf/rob_inmoov.xacro (robot description, xacro)
@@ -72,5 +72,5 @@
    <visual>
       <geometry>
-        <mesh filename="package://robbie_description/meshes/chest_cover.stl" scale="${M_SCALE} ${M_SCALE} ${M_SCALE}"/>
+        <mesh filename="package://robbie_description/meshes/chest_cover2.stl" scale="${M_SCALE} ${M_SCALE} ${M_SCALE}"/>
       </geometry>
          <xacro:gold/>
@@ -276,5 +276,5 @@
       </collision>
     </link>
-  <link name="head_cam_link">
+  <link name="camera_link">
       <inertial>
         <mass value="1.0" />
@@ -724,15 +724,15 @@
          </inertial>
       </link>
-  <joint name="head_cam_joint" type="fixed">
+  <joint name="camera_joint" type="fixed">
     	<parent link="head_link" />
-    	<child link="head_cam_link" />
+    	<child link="camera_link" />
     	<origin xyz="0.15 0.11 0.13" rpy="0 0.1 0" />
 	</joint>
-<joint name="head_cam_depth_joint" type="fixed">
+<joint name="camera_depth_joint" type="fixed">
          <origin xyz="0 0.0125 0.015" rpy="0 0 0" />
-          <parent link="head_cam_link" />
-          <child link="head_cam_depth_frame" />
+          <parent link="camera_link" />
+          <child link="camera_depth_frame" />
       </joint>
-      <link name="head_cam_depth_frame">
+      <link name="camera_depth_frame">
       <inertial>
          <mass value="0.000001" />
@@ -743,10 +743,10 @@
          </inertial>
       </link>
-      <joint name="head_cam_depth_optical_joint" type="fixed">
+      <joint name="camera_depth_optical_joint" type="fixed">
          <origin xyz="0 0 0" rpy="${-PI/2} 0 ${-PI/2}" />
-         <parent link="head_cam_depth_frame" />
-         <child link="head_cam_depth_optical_frame" />
+         <parent link="camera_depth_frame" />
+         <child link="camera_depth_optical_frame" />
       </joint>
-      <link name="head_cam_depth_optical_frame">
+      <link name="camera_depth_optical_frame">
          <inertial>
             <mass value="0.000001" />
@@ -757,10 +757,10 @@
          </inertial>
       </link>
-      <joint name="head_cam_rgb_joint" type="fixed">
+      <joint name="camera_rgb_joint" type="fixed">
          <origin xyz="0 -0.0125 0.015" rpy="0 0 0" />
-         <parent link="head_cam_link" />
-         <child link="head_cam_rgb_frame" />
+         <parent link="camera_link" />
+         <child link="camera_rgb_frame" />
       </joint>
-      <link name="head_cam_rgb_frame">
+      <link name="camera_rgb_frame">
          <inertial>
          <mass value="0.000001" />
@@ -771,10 +771,10 @@
          </inertial>
       </link>
-      <joint name="head_cam_rgb_optical_joint" type="fixed">
+      <joint name="camera_rgb_optical_joint" type="fixed">
          <origin xyz="0 0 0" rpy="${-PI/2} 0 ${-PI/2}" />
-         <parent link="head_cam_rgb_frame" />
-         <child link="head_cam_rgb_optical_frame" />
+         <parent link="camera_rgb_frame" />
+         <child link="camera_rgb_optical_frame" />
       </joint>
-      <link name="head_cam_rgb_optical_frame">
+      <link name="camera_rgb_optical_frame">
          <inertial>
             <mass value="0.000001" />
